Commit message: setup ros2-control for gazebo

File: vector_description/urdf/vector_arm.urdf.xacro (robot description, xacro)
@@ -3,4 +3,6 @@
     <xacro:include filename="$(find vector_description)/urdf/materials.xacro"/>
     <xacro:include filename="$(find vector_description)/urdf/vector_arm_macro.xacro"/>
+    <xacro:include filename="$(find vector_description)/urdf/vector_arm_ros2_control.xacro"/>
     <xacro:vector_arm prefix=""/>
+    <xacro:vector_arm_ros2_control prefix=""/>
 </robot>

File: vector_description/urdf/vector_arm_macro.xacro (robot description, xacro)
@@ -2,4 +2,5 @@
 <robot xmlns:xacro="http://www.ros.org/wiki/xacro">
     <xacro:macro name="vector_arm" params="prefix">
+        <link name="${prefix}world"/>
         <link name="${prefix}base_link">
             <visual>
@@ -325,5 +326,9 @@
             <parent link="${prefix}gripper_link"/>
             <child link="${prefix}gripper_frame_link"/>
-            <axis xyz="0 0 0"/>
+        </joint>
+        <joint name="${prefix}world_to_base" type="fixed">
+            <origin xyz="0 0 0" rpy="0 0 0"/>
+            <parent link="${prefix}world"/>
+            <child link="${prefix}base_link"/>
         </joint>
     </xacro:macro>
